Commit message: feat: no more errors

File: urdf/slam_bot.xacro (robot description, xacro)
@@ -153,4 +153,13 @@
     <parent link="chassis" />
   </joint>
+ <!--
+  <link name = "camera_rgbd_frame">
+  </link>
+  <joint type = "fixed" name ="camera_rgbd_joint">
+	<origin xyz="0 0 0" />
+	<child link ="camera_rgbd_frame" />
+	<parent link ="camera_link" />
+  </joint>
+  -->
 <!--LIDAR-->
 <link name="hokuyo">

Commit message: feat: slam mapping works. map made.

File: urdf/slam_bot.xacro (robot description, xacro)
@@ -153,14 +153,10 @@
     <parent link="chassis" />
   </joint>
- <!--
-  <link name = "camera_rgbd_frame">
+  <link name="camera_rgbd_frame">
   </link>
-  <joint type = "fixed" name ="camera_rgbd_joint">
-	<origin xyz="0 0 0" />
-	<child link ="camera_rgbd_frame" />
-	<parent link ="camera_link" />
+  <joint type="fixed" name="camera_rgbd_frame_joint">
+    <child link="camera_rgbd_frame" />
+    <parent link="camera" />
   </joint>
-  -->
-<!--LIDAR-->
 <link name="hokuyo">
     <origin>0. 0 0 0 0 0</origin>

Commit message: feat: kitchen dining fully mapped

File: urdf/slam_bot.xacro (robot description, xacro)
@@ -156,4 +156,5 @@
   </link>
   <joint type="fixed" name="camera_rgbd_frame_joint">
+	  <origin xyz="0 0 0" rpy="-1.57 0 -1.57" />
     <child link="camera_rgbd_frame" />
     <parent link="camera" />
